Commit message: Add farmer in simulation
- move base only works with mirte rn

File: bullproof_ws/src/mirte-ros-packages/mirte_description/urdf/farmer.urdf.xacro (robot description, xacro)
@@ -1,4 +1,4 @@
 <?xml version="1.0"?>
-<robot xmlns:xacro="http://www.ros.org/wiki/xacro" name="mirte">
+<robot xmlns:xacro="http://www.ros.org/wiki/xacro" name="farmer">
   <xacro:property name="package_name" value="mirte_description"/>
   <xacro:property name="robot_name" value="mirte"/>
@@ -20,5 +20,5 @@
   <xacro:footprint wheel_props="${front_wheel_props}" />
   <!-- Base link -->
-  <xacro:base base_prop="${base_props}" mesh="${base_props['base']['mesh']}" gazebo_color="Gazebo/White" rviz_color="white">
+  <xacro:base base_prop="${base_props}" mesh="${base_props['base']['mesh']}" gazebo_color="Gazebo/Red" rviz_color="red">
     <origin xyz="0 0 0" rpy="0 0 0" />
   </xacro:base>
@@ -46,10 +46,10 @@
   </xacro:motor>
   <!-- Sensors -->
-  <xacro:laser prefix="rplidar" parent_link="base_link"
+  <!-- <xacro:laser prefix="rplidar" parent_link="base_link"
                    sensor_prop="${sensor_prop}"
                    enable_gpu="${sensor_prop['laser']['enable_gpu']}">
-  </xacro:laser>
+  </xacro:laser> -->
   <!-- Gazebo -->
-  <xacro:gazebo_ros_control robotNamespace="/mirte">
+  <xacro:gazebo_ros_control robotNamespace="/farmer">
   </xacro:gazebo_ros_control>
 </robot>

File: bullproof_ws/src/mirte-ros-packages/mirte_description/urdf/include/common_macros.urdf.xacro (robot description, xacro)
@@ -156,5 +156,5 @@
 -->
   <xacro:macro name="base"
-               params="base_prop mesh:='' scale:='' *origin ">
+               params="base_prop mesh:='' scale:='' *origin gazebo_color rviz_color">
     <link name="base_link">
     <xacro:box_inertia m="${base_prop['base']['mass']}"
@@ -175,5 +175,5 @@
           </xacro:if>
         </geometry>
-        <material name="white" />
+        <material name="${rviz_color}" />
       </visual>
     </xacro:if>
@@ -184,5 +184,5 @@
           <box size="${base_prop['base']['x_size']} ${base_prop['base']['y_size']} ${base_prop['base']['z_size']}"/>
         </geometry>
-        <material name="white" />
+        <material name="${rviz_color}" />
       </visual>
     </xacro:if>
@@ -194,4 +194,7 @@
     </collision>
     </link>
+    <gazebo reference="base_link">
+      <material>${gazebo_color}</material>
+    </gazebo>
   </xacro:macro>
 <!-- ===================== Footprint xacro ==========================================

File: bullproof_ws/src/mirte-ros-packages/mirte_description/urdf/include/robot.gazebo.xacro (robot description, xacro)
@@ -3,5 +3,5 @@
   <!-- ros_control plugin -->
   <xacro:macro name="gazebo_ros_control" params="robotNamespace robotSimType:=gazebo_ros_control/DefaultRobotHWSim">
-    <gazebo>
+    <gazebo>etection algo
       <plugin name="p3d_base_controller" filename="libgazebo_ros_p3d.so">
         <alwaysOn>true</alwaysOn>
@@ -11,6 +11,9 @@
         <gaussianNoise>0.0</gaussianNoise>
         <frameName>map</frameName>
+        <!-- <frameId>/map -->
         <xyzOffsets>0 0 0</xyzOffsets>
         <rpyOffsets>0 0 0</rpyOffsets>
+        <!-- <namespace>"/"</namespace> -->
+        <!-- <robotNamespace>"/"</robotNamespace> -->
       </plugin>
       <plugin name="gazebo_ros_control" filename="libgazebo_ros_control.so">
